File: Hardware/CameraSlider/CameraSlider.sch (KiCad schematic (older format))
At the start: 19 parts, among them J1 Screw_Terminal_01x02, J10 Conn_01x04_Male, J11 Conn_01x04_Male, J2 Conn_01x02_Male, J3 Conn_01x03_Male, J4 Conn_01x02_Male, J5 Conn_01x02_Male, J6 Conn_01x03_Male, J7 Conn_01x03_Male, J8 Conn_02x03_Odd_Even, J9 Conn_01x04_Male, U1 A000005, U2 A4988_STEPPER_MOTOR_DRIVER_CA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

Commit message: Layout hinzugefügt
Connections:
- net at J11.1 (Pin_1): now also U2.14 (2B); no longer U2.12 (1A)
- net at J11.2 (Pin_2): now also U2.13 (2A); no longer U2.11 (1B)
- net at J11.3 (Pin_3): now also U2.11 (1B); no longer U2.13 (2A)
- net at J11.4 (Pin_4): now also U2.12 (1A); no longer U2.14 (2B)
Changed lines of the file:
@@
 L Connector:Conn_01x04_Male J11
 U 1 1 60CEF8B5
-P 9550 2150
-F 0 "J11" H 9522 2124 50  0000 R CNN
-F 1 "Conn_01x04_Male" H 9522 2033 50  0000 R CNN
-F 2 "Pin_Headers:Pin_Header_Angled_1x04_Pitch2.54mm" H 9550 2150 50  0001 C CNN
-F 3 "~" H 9550 2150 50  0001 C CNN
-	1    9550 2150
-	-1   0    0    -1
+P 9550 2250
+F 0 "J11" H 9522 2224 50  0000 R CNN
+F 1 "Conn_01x04_Male" H 9522 2133 50  0000 R CNN
+F 2 "Pin_Headers:Pin_Header_Angled_1x04_Pitch2.54mm" H 9550 2250 50  0001 C CNN
+F 3 "~" H 9550 2250 50  0001 C CNN
+	1    9550 2250
+	-1   0    0    1
 $EndComp
 Wire Wire Line
